File: pcb/esp32-rf-tools.kicad_sch (KiCad schematic)
At the start: 0 parts

Commit message: Add TP4056 module symbol and first schematic/PCB placement
- New symbol TP4056_Module_Protected (own work), linked to the
  matching footprint; provenance row in lib/README.md
- Schematic: ESP32-WROOM-32UE (U1), NRF24L01_Breakout (U2) and
  DLS24035B LCD (DS1) placed
- PCB: their footprints (nRF24 as nRF24L01_PA_LNA_SMA) and board
  outline
- .gitignore for KiCad lock files, local history, backups and caches

Co-Authored-By: Claude Opus 5 <noreply@anthropic.com>
Claude-Session: https://claude.ai/code/session_01F4q1FdRzA8RPNZWMDdwP16
Parts:
- added DS1: DLS24035B, esp32-rf-tools:DLS24035B, symbol esp32-rf-tools:DLS24035B
- added U1: ESP32-WROOM-32UE, esp32-rf-tools:ESP32-WROOM-32UE, symbol esp32-rf-tools:ESP32-WROOM-32UE
- added U2: NRF24L01_Breakout, esp32-rf-tools:nRF24L01_PA_LNA_SMA, symbol esp32-rf-tools:NRF24L01_Breakout
Connections:
- new net: U1.1 (GND), U1.15 (GND), U1.38 (GND)
