File: pcb/esp32-rf-tools.kicad_sch (KiCad schematic)
At the start: 3 parts, among them U1 ESP32-WROOM-32UE, U2 NRF24L01_Breakout

Commit message: m1
Parts:
- added D1: LED, LED_THT:LED_D5.0mm, symbol Device:LED
- added U3: TP4056_Module_Protected, esp32-rf-tools:TP4056_Module_Protected, symbol esp32-rf-tools:TP4056_Module_Protected
- added U4: CC1101, esp32-rf-tools:CC1101, symbol esp32-rf-tools:CC1101
- added U5: NRF24L01_Breakout, esp32-rf-tools:nRF24L01_PA_LNA_SMA, symbol esp32-rf-tools:NRF24L01_Breakout

Commit message: m2
Parts:
- removed U1: ESP32-WROOM-32UE, esp32-rf-tools:ESP32-WROOM-32UE, symbol esp32-rf-tools:ESP32-WROOM-32UE
- removed U4: CC1101, esp32-rf-tools:CC1101, symbol esp32-rf-tools:CC1101
- added BATT1: Battery 3.7v 550mAh, truke:Battery 902030, symbol truke:battery_3.7v_550mAh
- added U1: Step-up 3.7 - 12V, truke:Step-up_3.7_12, symbol truke:Step-up_3.7-12V
- added U4: (no value), truke:CC1101 433 MHz, symbol truke:CC1101_433MHz
- added U6: ESP32-DevKitC, PCM_Espressif:ESP32-DevKitC, symbol PCM_Espressif:ESP32-DevKitC
Connections:
- new net: U6.14 (GND), U6.32 (GND), U6.38 (GND)

Commit message: m3
Parts:
- added D2: D_Photo, LED_THT:LED_D5.0mm, symbol Device:D_Photo
- added SW1, SW2, SW3, SW4: SW_Push, Button_Switch_THT:SW_PUSH_6mm, symbol Switch:SW_Push
