File: pcb/esp32-rf-tools.kicad_pcb (KiCad board)
At the start: 2 copper layers, 120 x 75 mm, 3 parts, among them U1 ESP32-WROOM-32UE, U2 NRF24L01_Breakout

Commit message: m1
Parts:
- added D1: LED, LED_THT:LED_D5.0mm, F.Cu at (177.0, 68.2)
- added U3: TP4056_Module_Protected, esp32-rf-tools:TP4056_Module_Protected, F.Cu at (150.0, 60.0)
- added U4: CC1101, esp32-rf-tools:CC1101, F.Cu at (179.5, 37.0)
- added U5: NRF24L01_Breakout, esp32-rf-tools:nRF24L01_PA_LNA_SMA, F.Cu at (116.2, 86.8)

Commit message: m2
Parts:
- added BATT1: Battery 3.7v 550mAh, truke:Battery 902030, F.Cu at (101.1, 114.7)
- added U4: ~, truke:CC1101 433 MHz, F.Cu at (129.6, 50.8)
- added U6: ESP32-DevKitC, PCM_Espressif:ESP32-DevKitC, F.Cu at (124.5, 76.6)
- U1: value ESP32-WROOM-32UE -> Step-up 3.7 - 12V; footprint esp32-rf-tools:ESP32-WROOM-32UE -> truke:Step-up_3.7_12
- moved U3 55.7 mm to (167.1, 113.0)
- moved U5 45.1 mm to (161.3, 87.9)
- moved U1 38.5 mm to (161.8, 102.5)
- moved DS1 3.77 mm to (182.9, 71.1)
- moved U2 2.24 mm to (97.8, 87.9)
Connections:
- U1 pad 1: Net-(U1-GND-Pad1) -> unconnected-(U1-IN+-Pad1)

Commit message: m3
Parts:
- removed the U4 at (179.5, 37.0)
- added D2: D_Photo, LED_THT:LED_D5.0mm, F.Cu at (128.5, 54.6)
- added SW1: SW_Push, Button_Switch_THT:SW_PUSH_6mm, F.Cu at (72.4, 68.3)
- added SW2: SW_Push, Button_Switch_THT:SW_PUSH_6mm, F.Cu at (72.4, 78.5)
- added SW3: SW_Push, Button_Switch_THT:SW_PUSH_6mm, F.Cu at (72.4, 88.9)
- added SW4: SW_Push, Button_Switch_THT:SW_PUSH_6mm, F.Cu at (72.4, 99.1)
- moved U1 42.1 mm to (120.7, 93.2), turned to 90 degrees
- moved D1 42.1 mm to (137.2, 54.6)
- moved BATT1 13.1 mm to (101.6, 101.6), turned to 0 degrees
- moved U3 10.3 mm to (165.1, 102.9), turned to 90 degrees
- moved U6 8.03 mm to (127.0, 69.0)
- moved U4 5.76 mm to (123.9, 50.3)
- moved DS1 3.81 mm to (179.1, 71.1)
- moved U2 3.78 mm to (94.2, 86.6)
- moved U5 1.37 mm to (160.8, 86.6)
Other:
- board size 120 x 75 mm -> 116 x 75 mm
